Commit message: Add wheels

File: my_robot/urdf/my_robot.xacro (robot description, xacro)
@@ -55,3 +55,57 @@
     </visual>
   </link>
+  <joint name="left_wheel_hinge" type="continuous">
+    <origin xyz="0.0 0.15 0.0" rpy="0.0 0.0 0.0"/>
+    <child link="left_wheel"/>
+    <parent link="chassis"/>
+    <axis xyz="0.0 1 0" rpy= "0 0 0"/>
+    <limit lower="0.0" upper="0.0" effort="10000" velocity="10000"/>
+    <dynamics damping="1.0" friction="1.0"/>
+  </joint>
+  <link name='left_wheel'>
+    <inertial>
+      <mass value="5"/>
+      <origin xyz="0.0 0.0 0.0" rpy="0.0 1.5707 1.5707"/>
+      <inertia ixx="0.1" ixy="0.0" ixz="0.0" iyy="0.1" iyz="0.0" izz="0.1"/>
+    </inertial>
+    <collision name='collision'>
+      <origin xyz="0.0 0.0 0.0" rpy="0.0 1.5707 1.5707"/>
+      <geometry>
+        <cylinder radius="0.1" length="0.05"/>
+      </geometry>
+    </collision>
+    <visual name='chassis_visual'>
+      <origin xyz="0.0 0.0 0.0" rpy="0.0 1.5707 1.5707"/>
+      <geometry>
+        <cylinder radius="0.1" length="0.05"/>
+      </geometry>
+    </visual>
+  </link>
+  <joint name="right_wheel_hinge" type="continuous">
+    <origin xyz="0.0 -0.15 0.0" rpy="0.0 0.0 0.0"/>
+    <child link="right_wheel"/>
+    <parent link="chassis"/>
+    <axis xyz="0.0 1 0" rpy= "0 0 0"/>
+    <limit lower="0.0" upper="0.0" effort="10000" velocity="10000"/>
+    <dynamics damping="1.0" friction="1.0"/>
+  </joint>
+  <link name='right_wheel'>
+    <inertial>
+      <mass value="5"/>
+      <origin xyz="0.0 0.0 0.0" rpy="0.0 1.5707 1.5707"/>
+      <inertia ixx="0.1" ixy="0.0" ixz="0.0" iyy="0.1" iyz="0.0" izz="0.1"/>
+    </inertial>
+    <collision name='collision'>
+      <origin xyz="0.0 0.0 0.0" rpy="0.0 1.5707 1.5707"/>
+      <geometry>
+        <cylinder radius="0.1" length="0.05"/>
+      </geometry>
+    </collision>
+    <visual name='chassis_visual'>
+      <origin xyz="0.0 0.0 0.0" rpy="0.0 1.5707 1.5707"/>
+      <geometry>
+        <cylinder radius="0.1" length="0.05"/>
+      </geometry>
+    </visual>
+  </link>
 </robot>

Commit message: Add camera

File: my_robot/urdf/my_robot.xacro (robot description, xacro)
@@ -96,5 +96,5 @@
       <inertia ixx="0.1" ixy="0.0" ixz="0.0" iyy="0.1" iyz="0.0" izz="0.1"/>
     </inertial>
-    <collision name='collision'>
+    <collision>
       <origin xyz="0.0 0.0 0.0" rpy="0.0 1.5707 1.5707"/>
       <geometry>
@@ -102,5 +102,5 @@
       </geometry>
     </collision>
-    <visual name='chassis_visual'>
+    <visual>
       <origin xyz="0.0 0.0 0.0" rpy="0.0 1.5707 1.5707"/>
       <geometry>
@@ -109,3 +109,28 @@
     </visual>
   </link>
+  <joint name="camera_joint" type="fixed">
+    <axis xyz="0.0 1 0.0"/>
+    <origin xyz="0.2 0.0 0.0" rpy="0.0 0.0 0.0"/>
+    <parent link="chassis"/>
+    <child link="camera"/>
+  </joint>
+  <link name="camera">
+    <inertial>
+      <origin xyz="0.0 0.0 0.0" rpy="0.0 0.0 0.0"/>
+      <mass value="0.1"/>
+      <inertia ixx="1e-6" ixy="0.0" ixz="0.0" iyy="1e-6" iyz="0.0" izz="1e-6"/>
+    </inertial>
+    <collision>
+      <origin xyz="0.0 0.0 0.0" rpy="0.0 0.0 0.0"/>
+      <geometry>
+        <box size="0.05 0.05 0.05"/>
+      </geometry>
+    </collision>
+    <visual>
+      <origin xyz="0.0 0.0 0.0" rpy="0.0 0.0 0.0"/>
+      <geometry>
+        <box size="0.05 0.05 0.05"/>
+      </geometry>
+    </visual>
+  </link>
 </robot>

Commit message: Add camera and LIDAR to the robot

File: my_robot/urdf/my_robot.xacro (robot description, xacro)
@@ -63,5 +63,5 @@
     <dynamics damping="1.0" friction="1.0"/>
   </joint>
-  <link name='left_wheel'>
+  <link name="left_wheel">
     <inertial>
       <mass value="5"/>
@@ -69,5 +69,5 @@
       <inertia ixx="0.1" ixy="0.0" ixz="0.0" iyy="0.1" iyz="0.0" izz="0.1"/>
     </inertial>
-    <collision name='collision'>
+    <collision>
       <origin xyz="0.0 0.0 0.0" rpy="0.0 1.5707 1.5707"/>
       <geometry>
@@ -75,5 +75,5 @@
       </geometry>
     </collision>
-    <visual name='chassis_visual'>
+    <visual>
       <origin xyz="0.0 0.0 0.0" rpy="0.0 1.5707 1.5707"/>
       <geometry>
@@ -90,5 +90,5 @@
     <dynamics damping="1.0" friction="1.0"/>
   </joint>
-  <link name='right_wheel'>
+  <link name="right_wheel">
     <inertial>
       <mass value="5"/>
@@ -134,3 +134,42 @@
     </visual>
   </link>
+  <joint name="hokuyo_joint" type="fixed">
+    <parent link="chassis"/>
+    <child link="hokuyo"/>
+    <origin xyz="0.15  0.0 0.05" rpy="0.0 0.0 0.0"/>
+  </joint>
+  <link name="hokuyo">
+    <visual>
+      <geometry>
+        <mesh filename="package://my_robot/meshes/hokuyo.dae"/>
+        <box size="0.1 0.1 0.1" />
+        <cylinder radius="1.0" length="1.0"/>
+      </geometry>
+    </visual>
+    <collision>
+      <geometry>
+        <mesh filename="package://my_robot/meshes/hokuyo.dae"/>
+        <box size="0.1 0.1 0.1" />
+        <cylinder radius="1.0" length="1.0"/>
+      </geometry>
+    </collision>
+    <inertial>
+      <mass value="1e-5"/>
+      <origin xyz="0.0 0.0 0.0" rpy="0.0 0.0 0.0"/>
+      <inertia ixx="1e6" ixy="0.0" ixz="0.0" iyy="1e6" iyz="0.0" izz="1e6"/>
+    </inertial>
+  </link>
+  <!-- coloring the robot -->
+  <gazebo reference="camera">
+    <material>Gazebo/Blue</material>
+  </gazebo>
+  <gazebo reference="left_wheel">
+    <material>Gazebo/Grey</material>
+  </gazebo>
+  <gazebo reference="right_wheel">
+    <material>Gazebo/Grey</material>
+  </gazebo>
+  <gazebo reference="chassis">
+    <material>Gazebo/Red</material>
+  </gazebo>
 </robot>

Commit message: Load rviz config

File: my_robot/urdf/my_robot.xacro (robot description, xacro)
@@ -172,5 +172,5 @@
   </gazebo>
   <gazebo reference="chassis">
-    <material>Gazebo/Red</material>
+    <material>Gazebo/Green</material>
   </gazebo>
 </robot>

Commit message: Add world map

File: my_robot/urdf/my_robot.xacro (robot description, xacro)
@@ -158,5 +158,5 @@
       <mass value="1e-5"/>
       <origin xyz="0.0 0.0 0.0" rpy="0.0 0.0 0.0"/>
-      <inertia ixx="1e6" ixy="0.0" ixz="0.0" iyy="1e6" iyz="0.0" izz="1e6"/>
+      <inertia ixx="1e-6" ixy="0.0" ixz="0.0" iyy="1e-6" iyz="0.0" izz="1e-6"/>
     </inertial>
   </link>

Commit message: First rtab configuration

File: my_robot/urdf/my_robot.xacro (robot description, xacro)
@@ -135,4 +135,14 @@
     </visual>
   </link>
+  <!-- RGB-D camera -->
+  <joint name="camera_optical_joint" type="fixed">
+    <origin xyz="0 0 0" rpy="-1.5707 0 -1.5707"/>
+    <!-- <parent link="chassis"/> -->
+    <parent link="camera"/>
+    <child link="camera_link_optical"/>
+  </joint>
+  <link name="camera_link_optical">
+  </link>
+  <!-- Hokuyo LIDAR -->
   <joint name="hokuyo_joint" type="fixed">
     <parent link="chassis"/>
